File: hardware/carrier/carrier.kicad_sch (KiCad schematic)
At the start: 14 parts, among them J1 Harness_4Runner, Q1 BUK7Y4R8-60E, Q2 BUK7Y4R8-60E, U1 LM74800-Q1

Commit message: Carrier schematic: 5 V buck, 3.3 V LDO, power hold, key sense, Pi header
Co-Authored-By: Claude Opus 5.5 <noreply@anthropic.com>
Claude-Session: https://claude.ai/code/session_01EoLoLi7g91W5u4w3UzwQgu
Parts:
- added C10, C11, C17, C18: 1uF, Capacitor_SMD:C_0603_1608Metric, symbol Device:C
- added C12, C16, C20, C21, C8, C9: 100nF, Capacitor_SMD:C_0603_1608Metric, symbol Device:C
- added C13: 22pF, Capacitor_SMD:C_0603_1608Metric, symbol Device:C
- added C14, C15, C19: 47uF, Capacitor_SMD:C_1210_3225Metric, symbol Device:C
- added C6, C7: 10uF, Capacitor_SMD:C_1206_3216Metric, symbol Device:C
- added D2, D3: 1N4148W, Diode_SMD:D_SOD-123, symbol Device:D
- added D4: BZT52C15, Diode_SMD:D_SOD-123, symbol Device:D_Zener
- added J2: Pi 4 GPIO, Connector_PinSocket_2.54mm:PinSocket_2x20_P2.54mm_Vertical, symbol carrier:RaspberryPi_GPIO_40
- added L1: 4.7uH, Inductor_SMD:L_Bourns_SRP1038C_10.0x10.0mm, symbol Device:L
- added Q3, Q4: MMBT3904, Package_TO_SOT_SMD:SOT-23, symbol Transistor_BJT:MMBT3904
- added R10: 24.9k, Resistor_SMD:R_0603_1608Metric, symbol Device:R_Small_US
- added R11, R13: 1k, Resistor_SMD:R_0603_1608Metric, symbol Device:R_Small_US
- added R12, R15, R18: 47k, Resistor_SMD:R_0603_1608Metric, symbol Device:R_Small_US
- added R14, R5, R9: 100k, Resistor_SMD:R_0603_1608Metric, symbol Device:R_Small_US
- added R16, R17, R19, R20: 10k, Resistor_SMD:R_0603_1608Metric, symbol Device:R_Small_US
- added R6: 26.7k, Resistor_SMD:R_0603_1608Metric, symbol Device:R_Small_US
- added R7: 33.2k, Resistor_SMD:R_0603_1608Metric, symbol Device:R_Small_US
- added R8: 0R, Resistor_SMD:R_0603_1608Metric, symbol Device:R_Small_US
- added U2: LM61460-Q1, carrier:TI_RJR0014A_VQFN-HR-14_3.5x4mm, symbol carrier:LM61460-Q1
- added U3: TLV75533PDBV, Package_TO_SOT_SMD:SOT-23-5, symbol Regulator_Linear:TLV75533PDBV
Connections:
- net +12V_PROT: now also C6.1, C7.1, C8.1, C9.1, R5.1, U2.[8,12] (VIN)
- net ACC_IN: now also D2.2 (A), R15.1
- net GND: now also C10.2, C11.2, C14.2, C15.2, C16.2, C17.2, C18.2, C19.2, C20.2, C21.2, C6.2, C7.2, C8.2, C9.2, D4.2 (A), J2.[20,25,30] (GND), J2.[34,39] (GND), J2.[6,9,14] (GND), Q3.2 (E), Q4.2 (E), R10.2, R14.2, R16.2, R19.2, R6.2, R7.2, U2.3 (AGND), U2.[9,11] (PGND), U3.2 (GND)
- net ILLUM_IN: now also R18.1
- net SYS_EN: now also C19.1, D3.1 (K), D4.1 (K), R12.2, R14.1
- new net: C12.1, R8.1, U2.14 (CBOOT)
- new net: R8.2, U2.13 (RBOOT)
- new net: C20.1, Q3.1 (B), R15.2, R16.1
- new net: C13.1, R11.2
- new net: C13.2, R10.1, R9.2, U2.4 (FB)
- new net: D2.1 (K), R12.1
- new net: C21.1, Q4.1 (B), R18.2, R19.1
- new net: R5.2, R6.1, U2.7 (EN/SYNC)
- new net: D3.2 (A), R13.2
- new net: C10.1, U2.2 (VCC)
- new net: C12.2, L1.1, U2.10 (SW)
- new net: R7.1, U2.6 (RT)
- new net +3V3: C18.1, R17.1, R20.1, U3.5 (OUT)
- new net +5V: C11.1, C14.1, C15.1, C16.1, C17.1, J2.[2,4] (5V), L1.2, R11.1, R9.1, U2.1 (BIAS), U3.1 (IN), U3.3 (EN)
- new net FAN1_PWM: J2.32 (GPIO12)
- new net FAN1_TACH: J2.36 (GPIO16)
- new net FAN2_PWM: J2.33 (GPIO13)
- new net FAN2_TACH: J2.7 (GPIO4)
- new net I2C_SCL: J2.5 (GPIO3)
- new net I2C_SDA: J2.3 (GPIO2)
- new net I2S_BCLK: J2.12 (GPIO18)
- new net I2S_DOUT: J2.40 (GPIO21)
- new net I2S_FSYNC: J2.35 (GPIO19)
- new net ID_SCL: J2.28 (ID_SC)
- new net ID_SDA: J2.27 (ID_SD)
- new net PI_HOLD: J2.37 (GPIO26), R13.1
- new net UART_RX: J2.10 (GPIO15)
- new net UART_TX: J2.8 (GPIO14)
- new net ~{ACC_ON}: J2.11 (GPIO17), Q3.3 (C), R17.2
- new net ~{ADC_ALERT}: J2.31 (GPIO6)
- new net ~{AMP_FAULT}: J2.18 (GPIO24)
- new net ~{AMP_MUTE}: J2.16 (GPIO23)
- new net ~{AMP_STBY}: J2.15 (GPIO22)
- new net ~{AMP_WARN}: J2.22 (GPIO25)
- new net ~{LIGHTS_ON}: J2.13 (GPIO27), Q4.3 (C), R20.2
- new net ~{RTC_INT}: J2.29 (GPIO5)
- no-connect marks 2 -> 11
Other:
- note added: "5 V BUCK: Pi, display, fans, 3.3 V"
- note added: "5V pins 2/4 carry Pi + display (~3 A): wide pour to the buck output."
- note added: "ACC alone holds SYS_EN ~5 s (100k x 47 uF) so a crank before the Pi boots doesn't drop power. BZT52C15 limits load dump on the cap."
- note added: "AGND ties to PGND at the IC only. Keep the VIN/PGND hot loop through the 100 nF caps tight (SNVSB70F 11.1)."
- note added: "GPIO2/3 already have 1.8k pull-ups on the Pi."
- note added: "Hung Pi: the BCM watchdog resets it, GPIO26 floats low (100k bleed), and the board powers off if the key is off."
- note added: "Key off: the Pi syncs and halts, SYS_EN decays under 1.13 V ~2 s later and the LM74800 cuts everything (3 uA standby)."
- note added: "PI_HOLD (GPIO26): config.txt gpio=26=op,dh raises it ~1 s after power-up; dtoverlay=gpio-poweroff drops it once the Pi halts."
- note added: "POWER HOLD + KEY / LIGHTS SENSE"
- note added: "Pi 3V3 (1/17) unused: the board makes its own +3V3."
- note added: "RASPBERRY PI 4 (40-pin, board underside)"
- note added: "VOUT = 1.0 V x (1 + 100k / 24.9k) = 5.02 V. Input ceramics 50 V X7R; the amp's PVDD bulk on +12V_PROT doubles as CIN-BLK."
- note added: "fSW 400 kHz (RT 33.2k), FPWM + spread spectrum. UVLO on 6.0 V / off 4.3 V (100k / 26.7k), rides through cranking dips."

Commit message: Carrier schematic: amplifier, output filters, SWC ADC, RTC, ID EEPROM, fans, MCLK option
Also fixes field justification on 180-degree fields in the schematic
writer and re-lays out the sheet so every section fits the A2 frame.
ERC is clean.

Co-Authored-By: Claude Opus 5.5 <noreply@anthropic.com>
Claude-Session: https://claude.ai/code/session_01EoLoLi7g91W5u4w3UzwQgu
Parts:
- removed D2, D3: 1N4148W, Diode_SMD:D_SOD-123, symbol Device:D
- removed D4: BZT52C15, Diode_SMD:D_SOD-123, symbol Device:D_Zener
- removed U2: LM61460-Q1, carrier:TI_RJR0014A_VQFN-HR-14_3.5x4mm, symbol carrier:LM61460-Q1
- removed U3: TLV75533PDBV, Package_TO_SOT_SMD:SOT-23-5, symbol Regulator_Linear:TLV75533PDBV
- added BT1: CR2032, Battery:BatteryHolder_Keystone_1060_1x2032, symbol Device:Battery_Cell
- added C22: 22pF, Capacitor_SMD:C_0603_1608Metric, symbol Device:C
- added C23, C24: 47uF, Capacitor_SMD:C_1210_3225Metric, symbol Device:C
- added C25, C28, C30, C32, C65: 100nF, Capacitor_SMD:C_0603_1608Metric, symbol Device:C
- added C26, C27, C35, C36, C37, C38: 1uF, Capacitor_SMD:C_0603_1608Metric, symbol Device:C
- added C29, C31, C33: 10uF, Capacitor_SMD:C_1206_3216Metric, symbol Device:C
- added C34, C41, C42, C43, C44, C45, C46, C47, C48, C49, C51, C53, C55, C57, C59, C61, C63: 1uF, Capacitor_SMD:C_0805_2012Metric, symbol Device:C
- added C39, C40: 2.2uF, Capacitor_SMD:C_0805_2012Metric, symbol Device:C
- added C50, C52, C54, C56, C58, C60, C62, C64: 1nF, Capacitor_SMD:C_0603_1608Metric, symbol Device:C
- added C66, C67: 18pF, Capacitor_SMD:C_0603_1608Metric, symbol Device:C
- added D2, D3: PESD5V0S1BL, Diode_SMD:D_SOD-323, symbol Device:D_TVS
- added D4, D5: 1N4148W, Diode_SMD:D_SOD-123, symbol Device:D
- added D6: BZT52C15, Diode_SMD:D_SOD-123, symbol Device:D_Zener
- added H1, H2, H3, H4: Pi, MountingHole:MountingHole_2.7mm_M2.5_Pad_Via, symbol Mechanical:MountingHole_Pad
- added H5, H6: Heatsink, MountingHole:MountingHole_3.2mm_M3_Pad_Via, symbol Mechanical:MountingHole_Pad
- added J3: UART, Connector_PinHeader_2.54mm:PinHeader_1x03_P2.54mm_Vertical, symbol Connector:Conn_01x03_Pin
- added JP1: EEPROM_WP, Jumper:SolderJumper-2_P1.3mm_Open_RoundedPad1.0x1.5mm, symbol Jumper:SolderJumper_2_Open
- added L2, L3, L4, L5, L6, L7, L8, L9: 3.3uH, Inductor_SMD:L_Wuerth_XHMI-6060, symbol Device:L
- added M1: FAN1, Connector:FanPinHeader_1x04_P2.54mm_Vertical, symbol Motor:Fan_4pin
- added M2: FAN2, Connector:FanPinHeader_1x04_P2.54mm_Vertical, symbol Motor:Fan_4pin
- added Q5, Q6: 2N7002, Package_TO_SOT_SMD:SOT-23, symbol Transistor_FET:2N7002
- added R21: 47k, Resistor_SMD:R_0603_1608Metric, symbol Device:R_Small_US
- added R22, R23, R31, R33: 10k, Resistor_SMD:R_0603_1608Metric, symbol Device:R_Small_US
- added R24, R28, R32, R34: 100k, Resistor_SMD:R_0603_1608Metric, symbol Device:R_Small_US
- added R25: 26.7k, Resistor_SMD:R_0603_1608Metric, symbol Device:R_Small_US
- added R26: 33.2k, Resistor_SMD:R_0603_1608Metric, symbol Device:R_Small_US
- added R27, R35, R36: 0R, Resistor_SMD:R_0603_1608Metric, symbol Device:R_Small_US
- added R29: 24.9k, Resistor_SMD:R_0603_1608Metric, symbol Device:R_Small_US
- added R30: 1k, Resistor_SMD:R_0603_1608Metric, symbol Device:R_Small_US
- added TP1: WP, TestPoint:TestPoint_Pad_D1.5mm, symbol Connector:TestPoint
- added U2: ADS1115IDGS, Package_SO:TSSOP-10_3x3mm_P0.5mm, symbol Analog_ADC:ADS1115IDGS
- added U3: DS3231SN, Package_SO:SOIC-16W_7.5x10.3mm_P1.27mm, symbol carrier:DS3231SN
- added U4: CAT24C32, Package_SO:SOIC-8_3.9x4.9mm_P1.27mm, symbol Memory_EEPROM:24LC32
- added U5: LM61460-Q1, carrier:TI_RJR0014A_VQFN-HR-14_3.5x4mm, symbol carrier:LM61460-Q1
- added U6: TLV75533PDBV, Package_TO_SOT_SMD:SOT-23-5, symbol Regulator_Linear:TLV75533PDBV
- added U7: TAS6424E-Q1, Package_SO:SSOP-56_7.5x18.5mm_P0.635mm, symbol carrier:TAS6424E-Q1
- added U8: CS2100-CP, Package_SO:MSOP-10_3x3mm_P0.5mm, symbol carrier:CS2100-CP
- added Y1: 12MHz, Crystal:Crystal_SMD_3225-4Pin_3.2x2.5mm, symbol Device:Crystal
- C10, C11, C17, C18: value 1uF -> 100nF
- C12: value 100nF -> 47uF; footprint Capacitor_SMD:C_0603_1608Metric -> Capacitor_SMD:C_1210_3225Metric
- C13: value 22pF -> 100nF
- C14: value 47uF -> 100nF; footprint Capacitor_SMD:C_1210_3225Metric -> Capacitor_SMD:C_0603_1608Metric
- C15: value 47uF -> 10uF; footprint Capacitor_SMD:C_1210_3225Metric -> Capacitor_SMD:C_1206_3216Metric
- C16: value 100nF -> 10uF; footprint Capacitor_SMD:C_0603_1608Metric -> Capacitor_SMD:C_1206_3216Metric
- C19: value 47uF -> 1uF; footprint Capacitor_SMD:C_1210_3225Metric -> Capacitor_SMD:C_0603_1608Metric
- C20: value 100nF -> 1uF
- C6, C7: value 10uF -> 100nF; footprint Capacitor_SMD:C_1206_3216Metric -> Capacitor_SMD:C_0603_1608Metric
- C8: value 100nF -> 10nF
- R10: value 24.9k -> 10k
- R11: value 1k -> 10k
- R12: value 47k -> 1k
- R13: value 1k -> 3.9k
- R14: value 100k -> 3.9k
- R16: value 10k -> 1k
- R17: value 10k -> 100k
- R5: value 100k -> 1k
- R6: value 26.7k -> 10k
- R7: value 33.2k -> 1k
- R8: value 0R -> 10k
- R9: value 100k -> 0R
Connections:
- net +12V_PROT: now also C15.1, C16.1, C17.1, C18.1, C28.1, C29.1, C30.1, C31.1, C32.1, C33.1, C34.1, R24.1, U5.[8,12] (VIN), U7.3 (VBAT), U7.[2,29,30] (PVDD), U7.[42,43] (PVDD), U7.[55,56] (PVDD); no longer C6.1, C7.1, C8.1, C9.1, R5.1
- net +3V3: now also C10.1, C11.1, C9.1, R10.1, R11.1, R12.1, R13.1, R14.1, R5.1, R7.1, C27.1, C35.1, C65.1, R23.1, R31.1, R33.1, U2.8 (VDD), U3.2 (VCC), U4.8 (VCC), U6.5 (OUT), U7.19 (VDD), U8.1 (VD); no longer C18.1, R17.1
- net +5V: now also C20.1, C23.1, C24.1, C25.1, C26.1, M1.2 (+), M2.2 (+), R28.1, R30.1, U5.1 (BIAS), U6.1 (IN), U6.3 (EN); no longer C11.1, C14.1, C15.1, C16.1, C17.1, R11.1, R9.1
- net ACC_IN: now also R18.1, D4.2 (A); no longer R15.1
- net BATT_MON: now also C8.1, U2.6 (AIN2)
- net FAN1_PWM: now also Q5.1 (G), R32.1
- net FAN1_TACH: now also M1.3 (Tacho), R31.2
- net FAN2_PWM: now also Q6.1 (G), R34.1
- net FAN2_TACH: now also M2.3 (Tacho), R33.2
- net GND: now also C12.2, C13.2, R17.2, R9.2, BT1.2 (-), C23.2, C24.2, C25.2, C26.2, C27.2, C28.2, C29.2, C30.2, C31.2, C32.2, C33.2, C34.2, C35.2, C39.2, C40.2, C49.2, C50.2, C51.2, C52.2, C53.2, C54.2, C55.2, C56.2, C57.2, C58.2, C59.2, C60.2, C61.2, C62.2, C63.2, C64.2, C65.2, C66.2, C67.2, D2.1 (A1), D3.1 (A1), D6.2 (A), H1.1, H2.1, H3.1, H4.1, H5.1, H6.1, J3.3 (Pin_3), JP1.2 (B), M1.1 (-), M2.1 (-), Q5.2 (S), Q6.2 (S), R22.2, R25.2, R26.2, R29.2, R32.2, R34.2, U2.1 (ADDR), U2.3 (GND), U2.7 (AIN3), U3.13 (GND), U3.[5,6,7,8] (GND), U3.[9,10,11,12] (GND), U4.1 (A0), U4.2 (A1), U4.3 (A2), U4.4 (GND), U5.3 (AGND), U5.[9,11] (PGND), U6.2 (GND), U7.16 (SDIN2), U7.22 (I2C_ADDR0), U7.23 (I2C_ADDR1), U7.[1,11,17] (GND), U7.[18,28,33] (GND), U7.[36,39,46] (GND), U7.[49,52] (GND), U8.2 (GND), U8.8 (AD0); no longer C21.2, R10.2, R14.2, R16.2, R6.2, R7.2
- net I2C_SCL: now also U2.10 (SCL), U3.16 (SCL), U7.20 (SCL), U8.9 (SCL)
- net I2C_SDA: now also U2.9 (SDA), U3.15 (SDA), U7.21 (SDA), U8.10 (SDA)
- net I2S_BCLK: now also R36.1, U7.13 (SCLK)
- net I2S_DOUT: now also U7.15 (SDIN1)
- net I2S_FSYNC: now also U7.14 (FSYNC), U8.5 (CLK_IN)
- net ID_SCL: now also R14.2, U4.6 (SCL)
- net ID_SDA: now also R13.2, U4.5 (SDA)
- net ILLUM_IN: now also R21.1; no longer R18.1
- net PI_HOLD: now also R16.1; no longer R13.1
- net SPK_FL+: now also C49.1, C50.1, L2.2
- net SPK_FL-: now also C51.1, C52.1, L3.2
- net SPK_FR+: now also C53.1, C54.1, L4.2
- net SPK_FR-: now also C55.1, C56.1, L5.2
- net SPK_RL+: now also C57.1, C58.1, L6.2
- net SPK_RL-: now also C59.1, C60.1, L7.2
- net SPK_RR+: now also C61.1, C62.1, L8.2
- net SPK_RR-: now also C63.1, C64.1, L9.2
- net SWC1_IN: now also R5.2, R6.1, D2.2 (A2)
- net SWC2_IN: now also R7.2, R8.1, D3.2 (A2)
- net SWC_GND: now also R9.1
- net SYS_EN: now also C12.1, R15.2, R17.1, D5.1 (K), D6.1 (K); no longer C19.1, R12.2, R14.1
- net UART_RX: now also J3.2 (Pin_2)
- net UART_TX: now also J3.1 (Pin_1)
- net ~{ACC_ON}: now also R20.2; no longer R17.2
- net ~{ADC_ALERT}: now also R10.2, U2.2 (ALERT/RDY)
- net ~{AMP_FAULT}: now also U7.26 (~{FAULT})
- net ~{AMP_MUTE}: now also U7.25 (~{MUTE})
- net ~{AMP_STBY}: now also U7.24 (~{STANDBY})
- net ~{AMP_WARN}: now also U7.27 (~{WARN})
- net ~{LIGHTS_ON}: now also R23.2; no longer R20.2
- net ~{RTC_INT}: now also R11.2, U3.3 (~{INT}/SQW)
- net SWC2_ADC: now reaches R8.2
- net SWC2_ADC: now also C7.1, U2.5 (AIN1)
- net at C13.1: now also Q3.1 (B), R18.2, R19.1; no longer R11.2
- net at L1.1: now also C21.2, U5.10 (SW); no longer C12.2
- new net: C46.1, U7.44 (BST_3M)
- new net: BT1.1 (+), U3.14 (VBAT)
- new net: JP1.1 (A), R12.2, TP1.1, U4.7 (WP)
- new net: C39.1, C40.1, U7.[9,10] (GVDD)
- new net: C45.1, U7.48 (BST_3P)
- new net: C36.1, C37.1, U7.4 (AREF)
- new net: C37.2, U7.6 (VCOM)
- new net: C14.1, Q4.1 (B), R21.2, R22.1
- new net: C22.1, R30.2
- new net: C22.2, R28.2, R29.1, U5.4 (FB)
- new net: R24.2, R25.1, U5.7 (EN/SYNC)
- new net: R35.1, U8.3 (CLK_OUT)
- new net: C41.1, U7.35 (BST_1P)
- new net: C21.1, R27.1, U5.14 (CBOOT)
- new net: R27.2, U5.13 (RBOOT)
- new net: C42.1, U7.31 (BST_1M)
- new net: C44.1, U7.37 (BST_2M)
- new net: R26.1, U5.6 (RT)
- new net: M1.4 (PWM), Q5.3 (D)
- new net: C43.1, U7.41 (BST_2P)
- new net: C36.2, U7.5 (VREG)
- new net: C48.1, U7.50 (BST_4M)
- new net: C47.1, U7.54 (BST_4P)
- new net: C38.1, U7.7 (AVSS)
- new net: C38.2, U7.8 (AVDD)
- new net: D4.1 (K), R15.1
- new net: D5.2 (A), R16.2
- new net: C19.1, U5.2 (VCC)
- new net: M2.4 (PWM), Q6.3 (D)
- new net AMP_FL+: C41.2, L2.1, U7.34 (OUT_1P)
- new net AMP_FL-: C42.2, L3.1, U7.32 (OUT_1M)
- new net AMP_FR+: C43.2, L4.1, U7.40 (OUT_2P)
- new net AMP_FR-: C44.2, L5.1, U7.38 (OUT_2M)
- new net AMP_MCLK: R35.2, R36.2, U7.12 (MCLK)
- new net AMP_RL+: C45.2, L6.1, U7.47 (OUT_3P)
- new net AMP_RL-: C46.2, L7.1, U7.45 (OUT_3M)
- new net AMP_RR+: C47.2, L8.1, U7.53 (OUT_4P)
- new net AMP_RR-: C48.2, L9.1, U7.51 (OUT_4M)
- new net SWC1_ADC: C6.1, R6.2, U2.4 (AIN0)
- new net XTI: C66.1, U8.7 (XTI/REF_CLK), Y1.1
- new net XTO: C67.1, U8.6 (XTO), Y1.2
- no-connect marks 11 -> 14
Other:
- note added: "AIN0/1: wheel ladders, learned in software (press each button once)."
- note added: "AIN2: battery voltage (VBAT / 11.9). I2C address 0x48."
- note added: "AMP MCLK SELECT (CS2100 option, not fitted)"
- note added: "AMPLIFIER: TAS6424E-Q1, 4 x BTL, TDM from the Pi"
- note added: "Bypass bank: one 10 uF + 100 nF pair at each PVDD group (2/29/30, 42/43, 55/56), 1 uF at VBAT. Ceramics 50 V X7R."
- note added: "CS2100 I2C address 0x4E."
- note added: "Channel 1..4 = FL, FR, RL, RR (the Pi's TDM slot order; remap in software)."
- note added: "DEBUG UART + MOUNTING"
- note added: "Default: R (I2S_BCLK) fitted, MCLK = SCLK in TDM. Option: fit U, Y, caps and the CLK_OUT 0R instead, remove the BCLK 0R."
- note added: "EEPROM: 0x50 on ID_SD/ID_SC, 3.9k pull-ups, WP 1k up. Bridge JP to reflash (HAT design guide)."
- note added: "FANS (2 x Noctua 5 V PWM)"
- note added: "Fan PWM inputs float high inside the fan: no Pi, full speed."
- note added: "HSSOP-56 thermal pad is on TOP: clamp a GND-bonded heatsink on it. AREF and AVSS are local returns, not GND."
- note added: "Inductors: 3.3 uH, Isat >= 6 A, DCR <= 50 mR (SLOSE73A 10.2.1.2.4). 1 uF 50 V X7R, 1 nF C0G."
- note added: "OUTPUT FILTERS (2.1 MHz PWM -> speakers)"
- note added: "OV cutoff = 1.23 V x (95.3k + 5.11k + 3.65k) / 3.65k = 35.1 V. BATT_MON = VBAT / 11.9 (to ADS1115 AIN2)."
- note added: "PWM from the Pi's hardware PWM (GPIO12/13) at 25 kHz, inverted by the FET. Tach: 2 pulses per turn."
- note added: "Pi holes and the amp heatsink screws bond the Pi, heatsink and board GND."
- note added: "RTC (DS3231SN + CR2032) + HAT ID EEPROM"
- note added: "RTC: kernel i2c-rtc,ds3231 overlay, 0x68. Keeps time with the key off; the Pi reads it at boot."
- note added: "STEERING WHEEL + BATTERY ADC (ADS1115)"
- note added: "TDM4 on SDIN1, 32-bit slots, SCLK = 128 fs; MCLK = SCLK is allowed in TDM (SLOSE73A 9.3.1.4), jumper-selected in the clock block."
- note added: "UART: 3.3 V, GPIO14/15 serial console."
- note added: "~{STANDBY} / ~{MUTE} have 100k internal pull-downs: the amp stays silent until the Pi's I2C init. I2C address 0x6A."
- note removed: "OV cutoff = 1.23 V x (R1+R2+R3)/R3 = 35.1 V. BATT_MON = VBAT / 11.9 (to ADS1115 AIN2)."

Commit message: Carrier schematic: add the 470 uF PVDD bulk capacitor
Co-Authored-By: Claude Opus 5.5 <noreply@anthropic.com>
Claude-Session: https://claude.ai/code/session_01EoLoLi7g91W5u4w3UzwQgu
Parts:
- removed C35: 1uF, Capacitor_SMD:C_0603_1608Metric, symbol Device:C
- added C35: 470uF, Capacitor_SMD:CP_Elec_10x12.5, symbol Device:C_Polarized
- added C68: 18pF, Capacitor_SMD:C_0603_1608Metric, symbol Device:C
- C39: value 2.2uF -> 1uF; footprint Capacitor_SMD:C_0805_2012Metric -> Capacitor_SMD:C_0603_1608Metric
- C41: value 1uF -> 2.2uF
- C50, C52, C54, C56, C58, C60, C62, C64: value 1nF -> 1uF; footprint Capacitor_SMD:C_0603_1608Metric -> Capacitor_SMD:C_0805_2012Metric
- C51, C53, C55, C57, C59, C61, C63: value 1uF -> 1nF; footprint Capacitor_SMD:C_0805_2012Metric -> Capacitor_SMD:C_0603_1608Metric
- C65: value 100nF -> 1nF; now fitted
- C66: value 18pF -> 100nF
Connections:
- net +12V_PROT: now also C35.1
- net +3V3: now also C36.1, C66.1; no longer C65.1
- net AMP_FL+: now also C42.2; no longer C41.2
- net AMP_FL-: now also C43.2; no longer C42.2
- net AMP_FR+: now also C44.2; no longer C43.2
- net AMP_FR-: now also C45.2; no longer C44.2
- net AMP_RL+: now also C46.2; no longer C45.2
- net AMP_RL-: now also C47.2; no longer C46.2
- net AMP_RR+: now also C48.2; no longer C47.2
- net AMP_RR-: now also C49.2; no longer C48.2
- net GND: now also C36.2, C41.2, C35.2, C68.2; no longer C39.2, C49.2
- net SPK_FL+: now also C51.1; no longer C49.1
- net SPK_FL-: now also C53.1; no longer C51.1
- net SPK_FR+: now also C55.1; no longer C53.1
- net SPK_FR-: now also C57.1; no longer C55.1
- net SPK_RL+: now also C59.1; no longer C57.1
- net SPK_RL-: now also C61.1; no longer C59.1
- net SPK_RR+: now also C63.1; no longer C61.1
- net SPK_RR-: now also C65.1; no longer C63.1
- net XTI: now also C67.1; no longer C66.1
- net XTO: now also C68.1; no longer C67.1
- net at U7.44 (BST_3M): now also C47.1; no longer C46.1
- net at C40.1, U7.[9,10] (GVDD): now also C41.1; no longer C39.1
- net at C45.1: now also U7.37 (BST_2M); no longer U7.48 (BST_3P)
- net at C37.1, U7.4 (AREF): now also C38.1; no longer C36.1
- net at C37.2: now also U7.5 (VREG); no longer U7.6 (VCOM)
- net at U7.35 (BST_1P): now also C42.1; no longer C41.1
- net at U7.31 (BST_1M): now also C43.1; no longer C42.1
- net at C44.1: now also U7.41 (BST_2P); no longer U7.37 (BST_2M)
- net at U7.50 (BST_4M): now also C49.1; no longer C48.1
- net at U7.54 (BST_4P): now also C48.1; no longer C47.1
- net at U7.7 (AVSS): now also C39.1; no longer C38.1
- net at C38.2: now also U7.6 (VCOM); no longer U7.8 (AVDD)
- new net: C46.1, U7.48 (BST_3P)
- new net: C39.2, U7.8 (AVDD)
Other:
- note added: "10 x 12.5 mm, 50 V, 105 C"

Commit message: Carrier: pick every part, add MPN/Manufacturer/LCSC fields
All fitted parts are in JLCPCB stock. Swaps made while picking:
100 V caps upstream of the load-dump cutoff, a C0G 1 nF in the speaker
filters, 15 V ESD diodes on the wheel inputs (survive a short to 12 V),
33 pF crystal load caps, and footprints matched to the chosen inductors
and coin cell holder. The debug UART header is left unfitted.

Co-Authored-By: Claude Opus 5.5 <noreply@anthropic.com>
Claude-Session: https://claude.ai/code/session_01EoLoLi7g91W5u4w3UzwQgu
Parts:
- BT1: footprint Battery:BatteryHolder_Keystone_1060_1x2032 -> Battery:BatteryHolder_MYOUNG_BS-07-A1BJ001_CR2032; LCSC (none) -> C2979167; MPN (none) -> BS-07-A1BJ001; Manufacturer (none) -> MYOUNG
- C1, C2: LCSC (none) -> C28233; MPN (none) -> CL21B104KCFNNNE; Manufacturer (none) -> Samsung Electro-Mechanics
- C10, C11, C13, C14, C17, C18, C21, C25, C28, C30, C32, C6, C66, C7, C9: LCSC (none) -> C14663; MPN (none) -> CC0603KRX7R9BB104; Manufacturer (none) -> YAGEO
- C12, C23, C24: LCSC (none) -> C90142; MPN (none) -> TMK325ABJ476MM-P; Manufacturer (none) -> Taiyo Yuden
- C15, C16, C29, C31, C33: LCSC (none) -> C89632; MPN (none) -> CL31B106KBHNNNE; Manufacturer (none) -> Samsung Electro-Mechanics
- C19, C20, C26, C27, C36, C37, C38, C39: LCSC (none) -> C5199872; MPN (none) -> CL10B105KB8NQNC; Manufacturer (none) -> Samsung Electro-Mechanics
- C22: LCSC (none) -> C1653; MPN (none) -> CL10C220JB8NNNC; Manufacturer (none) -> Samsung Electro-Mechanics
- C3: LCSC (none) -> C1729; MPN (none) -> CL21B223KBANNNC; Manufacturer (none) -> Samsung Electro-Mechanics
- C34, C42, C43, C44, C45, C46, C47, C48, C49, C50, C52, C54, C56, C58, C60, C62, C64: LCSC (none) -> C28323; MPN (none) -> CL21B105KBFNNNE; Manufacturer (none) -> Samsung Electro-Mechanics
- C35: LCSC (none) -> C55348714; MPN (none) -> KAT1H471M10130PDT; Manufacturer (none) -> KNSCHA
- C4: footprint Capacitor_SMD:C_0603_1608Metric -> Capacitor_SMD:C_0805_2012Metric; LCSC (none) -> C28233; MPN (none) -> CL21B104KCFNNNE; Manufacturer (none) -> Samsung Electro-Mechanics
- C40, C41: LCSC (none) -> C77081; MPN (none) -> GRM21BR71E225KE11L; Manufacturer (none) -> Murata
- C5: LCSC (none) -> C64705; MPN (none) -> CL10B224KB8NNNC; Manufacturer (none) -> Samsung Electro-Mechanics
- C51, C53, C55, C57, C59, C61, C63, C65: LCSC (none) -> C163508; MPN (none) -> CL10C102JB8NNNC; Manufacturer (none) -> Samsung Electro-Mechanics
- C67, C68: value 18pF -> 33pF; LCSC (none) -> C1663; MPN (none) -> CL10C330JB8NNNC; Manufacturer (none) -> Samsung Electro-Mechanics
- C8: LCSC (none) -> C57112; MPN (none) -> 0603B103K500NT; Manufacturer (none) -> FH
- D1: LCSC (none) -> C19077587; MPN (none) -> SMBJ33CA; Manufacturer (none) -> hongjiacheng
- D2, D3: value PESD5V0S1BL -> H15VND3B; LCSC (none) -> C20615813; MPN (none) -> H15VND3B; Manufacturer (none) -> hongjiacheng
- D4, D5: LCSC (none) -> C81598; MPN (none) -> 1N4148W; Manufacturer (none) -> ST(Semtech)
- D6: LCSC (none) -> C19077412; MPN (none) -> BZT52C15; Manufacturer (none) -> hongjiacheng
- H1, H2, H3, H4, H5, H6, JP1, TP1: now left out of the parts list
- J1: LCSC (none) -> C485576; MPN (none) -> 430452000; Manufacturer (none) -> Molex
- J2: LCSC (none) -> C7499354; MPN (none) -> ZX-PM2.54-2-20PY; Manufacturer (none) -> Megastar
- J3: now not fitted
- L1: footprint Inductor_SMD:L_Bourns_SRP1038C_10.0x10.0mm -> Inductor_SMD:L_APV_APH0840; LCSC (none) -> C54123781; MPN (none) -> APH0840T4R7MP; Manufacturer (none) -> APV
- L2, L3, L4, L5, L6, L7, L8, L9: footprint Inductor_SMD:L_Wuerth_XHMI-6060 -> Inductor_SMD:L_Chilisin_BMRx00060630; LCSC (none) -> C108294; MPN (none) -> MHCI06030-3R3M-R8; Manufacturer (none) -> Chilisin
- M1, M2: LCSC (none) -> C240840; MPN (none) -> 470531000; Manufacturer (none) -> Molex
- Q1, Q2: LCSC (none) -> C503619; MPN (none) -> BUK7Y4R8-60EX; Manufacturer (none) -> Nexperia
- Q3, Q4: LCSC (none) -> C20526; MPN (none) -> MMBT3904; Manufacturer (none) -> Changjing
- Q5, Q6: LCSC (none) -> C8545; MPN (none) -> 2N7002; Manufacturer (none) -> Changjing
- R1: LCSC (none) -> C22775; MPN (none) -> 0603WAF1000T5E; Manufacturer (none) -> UNI-ROYAL
- R10, R11, R19, R20, R22, R23, R31, R33, R6, R8: LCSC (none) -> C25804; MPN (none) -> 0603WAF1002T5E; Manufacturer (none) -> UNI-ROYAL
- R12, R16, R30, R5, R7: LCSC (none) -> C21190; MPN (none) -> 0603WAF1001T5E; Manufacturer (none) -> UNI-ROYAL
- R13, R14: LCSC (none) -> C23018; MPN (none) -> 0603WAF3901T5E; Manufacturer (none) -> UNI-ROYAL
- R15, R18, R21: LCSC (none) -> C25819; MPN (none) -> 0603WAF4702T5E; Manufacturer (none) -> UNI-ROYAL
- R17, R24, R28, R32, R34: LCSC (none) -> C25803; MPN (none) -> 0603WAF1003T5E; Manufacturer (none) -> UNI-ROYAL
- R2: LCSC (none) -> C2907078; MPN (none) -> FRC0603F9532TS; Manufacturer (none) -> FOJAN
- R25: LCSC (none) -> C2930082; MPN (none) -> FRC0603F2672TS; Manufacturer (none) -> FOJAN
- R26: LCSC (none) -> C2933200; MPN (none) -> FRC0603F3322TS; Manufacturer (none) -> FOJAN
- R27, R35, R36, R9: LCSC (none) -> C21189; MPN (none) -> 0603WAF0000T5E; Manufacturer (none) -> UNI-ROYAL
- R29: LCSC (none) -> C25962; MPN (none) -> 0603WAF2492T5E; Manufacturer (none) -> UNI-ROYAL
- R3: LCSC (none) -> C2933233; MPN (none) -> FRC0603F5111TS; Manufacturer (none) -> FOJAN
- R4: LCSC (none) -> C2930089; MPN (none) -> FRC0603F3651TS; Manufacturer (none) -> FOJAN
- U1: LCSC (none) -> C3215600; MPN (none) -> LM74800QDRRRQ1; Manufacturer (none) -> Texas Instruments
- U2: LCSC (none) -> C37593; MPN (none) -> ADS1115IDGSR; Manufacturer (none) -> Texas Instruments
- U3: LCSC (none) -> C9866; MPN (none) -> DS3231SN#T&R; Manufacturer (none) -> Analog Devices
- U4: LCSC (none) -> C81193; MPN (none) -> CAT24C32WI-GT3; Manufacturer (none) -> onsemi
- U5: LCSC (none) -> C2876600; MPN (none) -> LM61460AFSQRJRRQ1; Manufacturer (none) -> Texas Instruments
- U6: LCSC (none) -> C404027; MPN (none) -> TLV75533PDBVR; Manufacturer (none) -> Texas Instruments
- U7: LCSC (none) -> C4991409; MPN (none) -> TAS6424EQDKQRQ1; Manufacturer (none) -> Texas Instruments
- U8: LCSC (none) -> C2663267; MPN (none) -> CS2100CP-CZZR; Manufacturer (none) -> Cirrus Logic
- Y1: LCSC (none) -> C9002; MPN (none) -> X322512MSB4SI; Manufacturer (none) -> YXC
Other:
- note added: "UART: 3.3 V, GPIO14/15 serial console. Header not fitted: solder one on if needed."
- note removed: "UART: 3.3 V, GPIO14/15 serial console."
