File: hardware/carrier/carrier.kicad_sch (KiCad schematic)
At the start: 148 parts, among them J1 Harness_4Runner, J2 Pi 4 GPIO, J3 UART, M1 FAN1, M2 FAN2, Q1 BUK7Y4R8-60E, Q2 BUK7Y4R8-60E, Q3 MMBT3904, Q4 MMBT3904, Q5 2N7002, Q6 2N7002, U1 LM74800-Q1, U2 ADS1115IDGS, U3 DS3231SN, U4 CAT24C32, U5 LM61460-Q1, U6 TLV75533PDBV, U7 TAS6424E-Q1, U8 CS2100-CP, Y1 12MHz

Commit message: Carrier: add a reverse-gear input (harness pin 10 to GPIO20)
Same 12 V sense circuit as ACC and ILLUM, active low into the Pi, for
an automatic backup camera or a music duck while reversing.

Co-Authored-By: Claude Opus 5.5 <noreply@anthropic.com>
Claude-Session: https://claude.ai/code/session_01EoLoLi7g91W5u4w3UzwQgu
Parts:
- removed C35: 470uF, Capacitor_SMD:CP_Elec_10x12.5, symbol Device:C_Polarized
- removed C36: 1uF, Capacitor_SMD:C_0603_1608Metric, symbol Device:C
- removed Q5: 2N7002, Package_TO_SOT_SMD:SOT-23, symbol Transistor_FET:2N7002
- added C35: 1uF, Capacitor_SMD:C_0805_2012Metric, symbol Device:C
- added C36: 470uF, Capacitor_SMD:CP_Elec_10x12.5, symbol Device:C_Polarized
- added C69: 33pF, Capacitor_SMD:C_0603_1608Metric, symbol Device:C
- added Q5: MMBT3904, Package_TO_SOT_SMD:SOT-23, symbol Transistor_BJT:MMBT3904
- added Q7: 2N7002, Package_TO_SOT_SMD:SOT-23, symbol Transistor_FET:2N7002
- added R37: 100k, Resistor_SMD:R_0603_1608Metric, symbol Device:R_Small_US
- added R38, R39: 0R, Resistor_SMD:R_0603_1608Metric, symbol Device:R_Small_US
- C15, C29, C31, C33: value 10uF -> 100nF; footprint Capacitor_SMD:C_1206_3216Metric -> Capacitor_SMD:C_0603_1608Metric; LCSC C89632 -> C14663; MPN CL31B106KBHNNNE -> CC0603KRX7R9BB104; Manufacturer Samsung Electro-Mechanics -> YAGEO
- C17, C30, C32: value 100nF -> 10uF; footprint Capacitor_SMD:C_0603_1608Metric -> Capacitor_SMD:C_1206_3216Metric; LCSC C14663 -> C89632; MPN CC0603KRX7R9BB104 -> CL31B106KBHNNNE; Manufacturer YAGEO -> Samsung Electro-Mechanics
- C19, C26: value 1uF -> 100nF; LCSC C5199872 -> C14663; MPN CL10B105KB8NQNC -> CC0603KRX7R9BB104; Manufacturer Samsung Electro-Mechanics -> YAGEO
- C21, C28: value 100nF -> 1uF; LCSC C14663 -> C5199872; MPN CC0603KRX7R9BB104 -> CL10B105KB8NQNC; Manufacturer YAGEO -> Samsung Electro-Mechanics
- C22: value 22pF -> 100nF; LCSC C1653 -> C14663; MPN CL10C220JB8NNNC -> CC0603KRX7R9BB104; Manufacturer Samsung Electro-Mechanics -> YAGEO
- C23: value 47uF -> 22pF; footprint Capacitor_SMD:C_1210_3225Metric -> Capacitor_SMD:C_0603_1608Metric; LCSC C90142 -> C1653; MPN TMK325ABJ476MM-P -> CL10C220JB8NNNC; Manufacturer Taiyo Yuden -> Samsung Electro-Mechanics
- C25: value 100nF -> 47uF; footprint Capacitor_SMD:C_0603_1608Metric -> Capacitor_SMD:C_1210_3225Metric; LCSC C14663 -> C90142; MPN CC0603KRX7R9BB104 -> TMK325ABJ476MM-P; Manufacturer YAGEO -> Taiyo Yuden
- C34: value 1uF -> 10uF; footprint Capacitor_SMD:C_0805_2012Metric -> Capacitor_SMD:C_1206_3216Metric; LCSC C28323 -> C89632; MPN CL21B105KBFNNNE -> CL31B106KBHNNNE
- C40: value 2.2uF -> 1uF; footprint Capacitor_SMD:C_0805_2012Metric -> Capacitor_SMD:C_0603_1608Metric; LCSC C77081 -> C5199872; MPN GRM21BR71E225KE11L -> CL10B105KB8NQNC; Manufacturer Murata -> Samsung Electro-Mechanics
- C42: value 1uF -> 2.2uF; LCSC C28323 -> C77081; MPN CL21B105KBFNNNE -> GRM21BR71E225KE11L; Manufacturer Samsung Electro-Mechanics -> Murata
- C51, C53, C55, C57, C59, C61, C63, C65: value 1nF -> 1uF; footprint Capacitor_SMD:C_0603_1608Metric -> Capacitor_SMD:C_0805_2012Metric; LCSC C163508 -> C28323; MPN CL10C102JB8NNNC -> CL21B105KBFNNNE
- C52, C54, C56, C58, C60, C62, C64: value 1uF -> 1nF; footprint Capacitor_SMD:C_0805_2012Metric -> Capacitor_SMD:C_0603_1608Metric; LCSC C28323 -> C163508; MPN CL21B105KBFNNNE -> CL10C102JB8NNNC
- C66: value 100nF -> 1nF; LCSC C14663 -> C163508; MPN CC0603KRX7R9BB104 -> CL10C102JB8NNNC; Manufacturer YAGEO -> Samsung Electro-Mechanics; now fitted
- C67: value 33pF -> 100nF; LCSC C1663 -> C14663; MPN CL10C330JB8NNNC -> CC0603KRX7R9BB104; Manufacturer Samsung Electro-Mechanics -> YAGEO
- R24: value 100k -> 47k; LCSC C25803 -> C25819; MPN 0603WAF1003T5E -> 0603WAF4702T5E
- R25: value 26.7k -> 10k; LCSC C2930082 -> C25804; MPN FRC0603F2672TS -> 0603WAF1002T5E; Manufacturer FOJAN -> UNI-ROYAL
- R26: value 33.2k -> 10k; LCSC C2933200 -> C25804; MPN FRC0603F3322TS -> 0603WAF1002T5E; Manufacturer FOJAN -> UNI-ROYAL
- R27: value 0R -> 100k; LCSC C21189 -> C25803; MPN 0603WAF0000T5E -> 0603WAF1003T5E
- R28: value 100k -> 26.7k; LCSC C25803 -> C2930082; MPN 0603WAF1003T5E -> FRC0603F2672TS; Manufacturer UNI-ROYAL -> FOJAN
- R29: value 24.9k -> 33.2k; LCSC C25962 -> C2933200; MPN 0603WAF2492T5E -> FRC0603F3322TS; Manufacturer UNI-ROYAL -> FOJAN
- R30: value 1k -> 0R; LCSC C21190 -> C21189; MPN 0603WAF1001T5E -> 0603WAF0000T5E
- R31: value 10k -> 100k; LCSC C25804 -> C25803; MPN 0603WAF1002T5E -> 0603WAF1003T5E
- R32: value 100k -> 24.9k; LCSC C25803 -> C25962; MPN 0603WAF1003T5E -> 0603WAF2492T5E
- R33: value 10k -> 1k; LCSC C25804 -> C21190; MPN 0603WAF1002T5E -> 0603WAF1001T5E
- R34: value 100k -> 10k; LCSC C25803 -> C25804; MPN 0603WAF1003T5E -> 0603WAF1002T5E
- R35: value 0R -> 100k; LCSC C21189 -> C25803; MPN 0603WAF0000T5E -> 0603WAF1003T5E; now fitted
- R36: value 0R -> 10k; LCSC C21189 -> C25804; MPN 0603WAF0000T5E -> 0603WAF1002T5E
Connections:
- net +12V_PROT: now also C19.1, R27.1, C35.1, C36.1; no longer C15.1, C28.1, R24.1
- net +3V3: now also C28.1, C37.1, C67.1, R26.1, R34.1, R36.1; no longer C27.1, C66.1, R31.1, R33.1
- net +5V: now also C21.1, C27.1, R31.1, R33.1; no longer C20.1, C23.1, R28.1, R30.1
- net AMP_FL+: now also C43.2; no longer C42.2
- net AMP_FL-: now also C44.2; no longer C43.2
- net AMP_FR+: now also C45.2; no longer C44.2
- net AMP_FR-: now also C46.2; no longer C45.2
- net AMP_MCLK: now also R38.2, R39.2; no longer R35.2, R36.2
- net AMP_RL+: now also C47.2; no longer C46.2
- net AMP_RL-: now also C48.2; no longer C47.2
- net AMP_RR+: now also C49.2; no longer C48.2
- net AMP_RR-: now also C50.2; no longer C49.2
- net FAN1_PWM: now also Q6.1 (G), R35.1; no longer R32.1
- net FAN1_TACH: now also R34.2; no longer R31.2
- net FAN2_PWM: now also Q7.1 (G), R37.1; no longer Q6.1 (G), R34.1
- net FAN2_TACH: now also R36.2; no longer R33.2
- net GND: now also C21.2, C37.2, C42.2, R28.2, R35.2, C35.2, C36.2, C69.2, Q5.2 (E), Q7.2 (S), R37.2; no longer C23.2, C40.2, C50.2, R26.2, R34.2
- net I2S_BCLK: now also R39.1; no longer R36.1
- net SPK_FL+: now also C52.1; no longer C50.1
- net SPK_FL-: now also C54.1; no longer C52.1
- net SPK_FR+: now also C56.1; no longer C54.1
- net SPK_FR-: now also C58.1; no longer C56.1
- net SPK_RL+: now also C60.1; no longer C58.1
- net SPK_RL-: now also C62.1; no longer C60.1
- net SPK_RR+: now also C64.1; no longer C62.1
- net SPK_RR-: now also C66.1; no longer C64.1
- net XTI: now also C68.1; no longer C67.1
- net XTO: now also C69.1; no longer C68.1
- net at U5.6 (RT): now also R29.1; no longer R26.1
- net at U7.35 (BST_1P): now also C43.1; no longer C42.1
- net at U7.37 (BST_2M): now also C46.1; no longer C45.1
- net at L1.1, U5.10 (SW): now also C22.2; no longer C21.2
- net at R27.2: now also R28.1, U5.7 (EN/SYNC); no longer U5.13 (RBOOT)
- net at U5.2 (VCC): now also C20.1; no longer C19.1
- net at R24.2, R25.1: now also C15.1, Q5.1 (B); no longer U5.7 (EN/SYNC)
- net at C48.1: now also U7.44 (BST_3M); no longer U7.54 (BST_4P)
- net ~{REVERSE}: now reaches J2.38 (GPIO20)
- net ~{REVERSE}: now also R26.2, Q5.3 (C)
- net at U8.3 (CLK_OUT): now also R38.1; no longer R35.1
- net at U7.48 (BST_3P): now also C47.1; no longer C46.1
- net at C44.1: now also U7.31 (BST_1M); no longer U7.41 (BST_2P)
- net at C38.1, U7.4 (AREF): now also C39.1; no longer C37.1
- net at U7.5 (VREG): now also C38.2; no longer C37.2
- net at C22.1: now also R30.1, U5.14 (CBOOT); no longer R30.2
- net at U7.6 (VCOM): now also C39.2; no longer C38.2
- net at C41.1, U7.[9,10] (GVDD): now also C42.1; no longer C40.1
- net at M1.4 (PWM): now also Q6.3 (D)
- net at M2.4 (PWM): now also Q7.3 (D); no longer Q6.3 (D)
- net at U7.50 (BST_4M): now also C50.1; no longer C49.1
- net at U7.7 (AVSS): now also C40.1; no longer C39.1
- net at U7.8 (AVDD): now also C40.2; no longer C39.2
- new net: C45.1, U7.41 (BST_2P)
- new net: C49.1, U7.54 (BST_4P)
- new net: C23.1, R33.2
- new net: R30.2, U5.13 (RBOOT)
- new net: C23.2, R31.2, R32.1, U5.4 (FB)
- new net REV_IN: J1.10 (REV), R24.1
- no-connect marks 14 -> 13
Other:
- note added: "POWER HOLD + KEY / LIGHTS / REVERSE SENSE"
- note removed: "POWER HOLD + KEY / LIGHTS SENSE"

Commit message: Carrier: vertical harness connector, deterministic schematic UUIDs
The harness plug now faces straight out of the board (toward the
firewall): Molex 43045-2012, LCSC C485575. Symbol and pin UUIDs are
derived from the reference so the PCB stays linked across regenerations.

Co-Authored-By: Claude Opus 5.5 <noreply@anthropic.com>
Claude-Session: https://claude.ai/code/session_01EoLoLi7g91W5u4w3UzwQgu
Parts:
- J1: footprint Connector_Molex:Molex_Micro-Fit_3.0_43045-2000_2x10_P3.00mm_Horizontal -> Connector_Molex:Molex_Micro-Fit_3.0_43045-2012_2x10_P3.00mm_Vertical; LCSC C485576 -> C485575; MPN 430452000 -> 430452012
