File: hardware/carrier/carrier.kicad_sch (KiCad schematic)
At the start: 157 parts, among them J1 Harness_4Runner, J2 Pi 4 GPIO, J3 UART, M1 FAN1, M2 FAN2, Q1 BUK7Y4R8-60E, Q2 BUK7Y4R8-60E, Q3 MMBT3904, Q4 MMBT3904, Q5 MMBT3904, Q6 2N7002, Q7 2N7002, U1 LM74800-Q1, U2 ADS1115IDGS, U3 DS3231SN, U4 CAT24C32, U5 LM61460-Q1, U6 TLV75533PDBV, U7 TAS6424E-Q1, U8 PCM1808-Q1, X1 12.288MHz

Commit message: Carrier: mic input and status LEDs (board to be re-routed)
Mic: 3.5 mm jack J4 (PJ-320D) with electret bias from +3V3 (1k + 10 uF
filter, 2.2k), ESD and 1 nF at the jack, 1 uF into the PCM1808's VINL.
PCM1808 DOUT goes to the Pi's I2S input on GPIO20, so ~REVERSE moves to
GPIO7. The overlay adds a capture codec on the same link; carrierd and
the docs follow. Three red status LEDs: 12 V protected, 5 V, PI_HOLD.
Serial console enabled for J3.

Tooling: the maze router checks the stub from an exact pad point to its
first grid cell; 0.5 mm keepout bands around the cable slot and notch;
OUTLINE_SHIFT in place.py moves the outer edge after measuring; the build
keeps a copy of the board right after the autorouter import.

Co-Authored-By: Claude Opus 5.5 <noreply@anthropic.com>
Claude-Session: https://claude.ai/code/session_01EoLoLi7g91W5u4w3UzwQgu
Parts:
- added C73: 10uF, Capacitor_SMD:C_0805_2012Metric, symbol Device:C
- added C74: 1uF, Capacitor_SMD:C_0603_1608Metric, symbol Device:C
- added C75: 1nF, Capacitor_SMD:C_0603_1608Metric, symbol Device:C
- added D10, D8, D9: RED, LED_SMD:LED_0603_1608Metric, symbol Device:LED
- added D7: H15VND3B, Diode_SMD:D_SOD-323, symbol Device:D_TVS
- added J4: MIC, Connector_Audio:Jack_3.5mm_PJ320D_Horizontal, symbol Connector_Audio:AudioJack4
- added R41: 33R, Resistor_SMD:R_0603_1608Metric, symbol Device:R_Small_US
- added R42: 2.2k, Resistor_SMD:R_0603_1608Metric, symbol Device:R_Small_US
- added R43, R45, R46: 1k, Resistor_SMD:R_0603_1608Metric, symbol Device:R_Small_US
- added R44: 10k, Resistor_SMD:R_0603_1608Metric, symbol Device:R_Small_US
Connections:
- net +12V_PROT: now also R44.1
- net +3V3: now also R43.1
- net +5V: now also R45.1
- net GND: now also C73.2, C75.2, D10.1 (K), D7.1 (A1), D8.1 (K), D9.1 (K), J4.R1, J4.R2, J4.S
- net I2S_BCLK: now also R40.2; no longer R39.2
- net I2S_FSYNC: now also R41.2; no longer R40.2
- net PI_HOLD: now also R46.1
- net ~{REVERSE}: now also J2.26 (GPIO7); no longer J2.38 (GPIO20)
- net at R39.1: now also U8.9 (DOUT); no longer U8.8 (BCK)
- net MIC_IN: now reaches U8.13 (VINL)
- net MIC_IN: now also C74.2
- net at U8.7 (LRCK): now also R41.1; no longer R40.1
- new net: C73.1, R42.1, R43.2
- new net: D8.2 (A), R44.2
- new net: D10.2 (A), R46.2
- new net: R40.1, U8.8 (BCK)
- new net: D9.2 (A), R45.2
- new net I2S_DIN: J2.38 (GPIO20), R39.2
- new net MIC_T: C74.1, C75.1, D7.2 (A2), J4.T, R42.2
- no-connect marks 15 -> 12
Other:
- note added: "12V ~1 mA"
- note added: "5V ~3 mA"
- note added: "Keep MIC_T / MIC_IN short and over solid GND, away from the amp outputs."
- note added: "MIC INPUT: electret, 3.5 mm jack -> PCM1808"
- note added: "Mic on the tip; ring + sleeve to GND. ~1.2 V bias at 0.5 mA. PCM1808 has no PGA: gain in software."
- note added: "PI HOLD ~1 mA"
- note added: "Pi I2S = clock consumer (slave). MCLK 256 fs, BCK 64 fs, LRCK 48 kHz, one oscillator. PCM1808 ADC: mic on VINL, DOUT to the Pi."
- note added: "STATUS LEDS (12V IN / 5V / PI HOLD)"
- note removed: "Pi I2S = clock consumer (slave). MCLK 256 fs, BCK 64 fs, LRCK 48 kHz, one oscillator. PCM1808 ADC unused."
- moved on the sheet: R39, R40
