File: hardware/carrier/carrier.kicad_sch (KiCad schematic)
At the start: 171 parts, among them J1 Harness_4Runner, J2 Pi 4 GPIO, J3 UART, J4 MIC, M1 FAN1, M2 FAN2, Q1 BUK7Y4R8-60E, Q2 BUK7Y4R8-60E, Q3 MMBT3904, Q4 MMBT3904, Q5 MMBT3904, Q6 2N7002, Q7 2N7002, U1 LM74800-Q1, U2 ADS1115IDGS, U3 DS3231SN, U4 CAT24C32, U5 LM61460-Q1, U6 TLV75533PDBV, U7 TAS6424E-Q1, U8 PCM1808-Q1, X1 12.288MHz

Commit message: Carrier: pre-order fixes from simulation and a placement check
Placement file: JLC places each part by its own footprint, and 16 of ours
are drawn turned relative to KiCad's (SOT-23s, LFPAK56s, U2-U4, U6, U7,
J1, the fan headers and the CR2032 holder, which would have gone in
reversed). jlc_cpl.py now adds the rotation JLC needs and moves BT1 and J4
to JLC's footprint origin (BT1 was 3.8 mm off, J4 0.9 mm). check_cpl.py
fits JLC's footprints pad by pad and checks fab/carrier_cpl.csv: 0
mismatches (the previous file fails 18).

R15 47k -> 10k: with the key turned straight to START, the hold cap now
fills in time and the board rides through a crank (4.6 s worst case, was
0.5 s). R4 3.65k -> 3.74k: OV cutoff 32.6-36.0 V over tolerances, inside
the LM61460's 36 V limit (was up to 36.8 V). Both are value changes on the
existing footprints; the board was patched in place, not re-routed.

sim.py runs SPICE testbenches for every analog block in KiCad's bundled
ngspice (37 checks over tolerance corners, all pass). Schematic notes and
README now give the simulated timings. VERIFICATION.md has the full
report; order with 1 oz inner copper.
Parts:
- R15: value 47k -> 10k; LCSC C25819 -> C25804; MPN 0603WAF4702T5E -> 0603WAF1002T5E
- R4: value 3.65k -> 3.74k; LCSC C2930089 -> C2933210; MPN FRC0603F3651TS -> FRC0603F3741TS
Other:
- note added: "ACC alone holds SYS_EN 4.7-10 s (100k x 47 uF), even after 0.3 s of ACC, so an early crank keeps power. BZT52C15 clamps load dump."
- note added: "AIN2: battery voltage (VBAT / 11.8). I2C address 0x48."
- note added: "Key off: the Pi halts; SYS_EN falls under 1.13 V 3-5 s later (load off), under 0.3-0.93 V after 7-12 s (3 uA standby)."
- note added: "Mic on the tip; ring + sleeve to GND. Bias 1.6-2.6 V (0.5-0.2 mA capsule). PCM1808 has no PGA: gain in software."
- note added: "OV cutoff = 1.23 V x (95.3k + 5.11k + 3.74k) / 3.74k = 34.3 V (32.6-36.0 V worst case). BATT_MON = VBAT / 11.8 (to ADS1115 AIN2)."
- note removed: "ACC alone holds SYS_EN ~5 s (100k x 47 uF) so a crank before the Pi boots doesn't drop power. BZT52C15 limits load dump on the cap."
- note removed: "AIN2: battery voltage (VBAT / 11.9). I2C address 0x48."
- note removed: "Key off: the Pi syncs and halts, SYS_EN decays under 1.13 V ~2 s later and the LM74800 cuts everything (3 uA standby)."
- note removed: "Mic on the tip; ring + sleeve to GND. ~1.2 V bias at 0.5 mA. PCM1808 has no PGA: gain in software."
- note removed: "OV cutoff = 1.23 V x (95.3k + 5.11k + 3.65k) / 3.65k = 35.1 V. BATT_MON = VBAT / 11.9 (to ADS1115 AIN2)."
