File: hardware/carrier/carrier.kicad_pcb (KiCad board)
At the start: 4 copper layers, 164.9 x 102 mm, 171 parts, among them J1 Harness_4Runner, J2 Pi 4 GPIO, J3 UART, J4 MIC, M1 FAN1, M2 FAN2, Q1 BUK7Y4R8-60E, Q2 BUK7Y4R8-60E, Q3 MMBT3904, Q4 MMBT3904, Q5 MMBT3904, Q6 2N7002, Q7 2N7002, U1 LM74800-Q1, U2 ADS1115IDGS, U3 DS3231SN, U4 CAT24C32, U5 LM61460-Q1, U6 TLV75533PDBV, U7 TAS6424E-Q1, U8 PCM1808-Q1, X1 12.288MHz

Commit message: Carrier: pre-order fixes from simulation and a placement check
Placement file: JLC places each part by its own footprint, and 16 of ours
are drawn turned relative to KiCad's (SOT-23s, LFPAK56s, U2-U4, U6, U7,
J1, the fan headers and the CR2032 holder, which would have gone in
reversed). jlc_cpl.py now adds the rotation JLC needs and moves BT1 and J4
to JLC's footprint origin (BT1 was 3.8 mm off, J4 0.9 mm). check_cpl.py
fits JLC's footprints pad by pad and checks fab/carrier_cpl.csv: 0
mismatches (the previous file fails 18).

R15 47k -> 10k: with the key turned straight to START, the hold cap now
fills in time and the board rides through a crank (4.6 s worst case, was
0.5 s). R4 3.65k -> 3.74k: OV cutoff 32.6-36.0 V over tolerances, inside
the LM61460's 36 V limit (was up to 36.8 V). Both are value changes on the
existing footprints; the board was patched in place, not re-routed.

sim.py runs SPICE testbenches for every analog block in KiCad's bundled
ngspice (37 checks over tolerance corners, all pass). Schematic notes and
README now give the simulated timings. VERIFICATION.md has the full
report; order with 1 oz inner copper.
Parts:
- R15: value 47k -> 10k
- R4: value 3.65k -> 3.74k
Changed lines of the file:
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@@
 			)
 		)
-		(property "Value" "47k"
+		(property "Value" "10k"
 			(at 0 1.43 0)
 			(layer "F.Fab")
@@
 			)
 		)
-		(property "LCSC" "C25819"
-			(at 0 0 0)
-			(layer "F.SilkS")
-			(hide yes)
-			(effects
-				(font
-					(size 1.27 1.27)
-					(thickness 0.15)
-				)
-			)
-		)
-		(property "MPN" "0603WAF4702T5E"
+		(property "LCSC" "C25804"
+			(at 0 0 0)
+			(layer "F.SilkS")
+			(hide yes)
+			(effects
+				(font
+					(size 1.27 1.27)
+					(thickness 0.15)
+				)
+			)
+		)
+		(property "MPN" "0603WAF1002T5E"
 			(at 0 0 0)
 			(layer "F.SilkS")
@@
 			)
 		)
-		(property "Value" "3.65k"
+		(property "Value" "3.74k"
 			(at 0 1.43 0)
 			(layer "F.Fab")
@@
 			)
 		)
-		(property "LCSC" "C2930089"
-			(at 0 0 0)
-			(layer "F.SilkS")
-			(hide yes)
-			(effects
-				(font
-					(size 1.27 1.27)
-					(thickness 0.15)
-				)
-			)
-		)
-		(property "MPN" "FRC0603F3651TS"
-			(at 0 0 0)
-			(layer "F.SilkS")
+		(property "LCSC" "C2933210"
+			(at 0 0 0)
+			(layer "F.SilkS")
+			(hide yes)
+			(effects
+				(font
+					(size 1.27 1.27)
+					(thickness 0.15)
+				)
+			)
+		)
+		(property "MPN" "FRC0603F3741TS"
+			(at 0 0 0)
+			(layer "F.SilkS")
